File: UINIO-MCU-STM32F103C8T6.kicad_sch (KiCad schematic)
At the start: 37 parts, among them J1 Conn_01x24_Pin, J2 Conn_01x24_Pin, J3 Conn_01x04_Pin, SW1 BOOT1, SW2 NRST, SW3 BOOT0, U1 ME6211C33M5G-N, U2 GD32F103C8T6, Y1 32.768KHz, Y2 8MHz

Commit message: Complete wiring.
Parts:
- removed R7: 1M, Resistor_SMD:R_0402_1005Metric, symbol Device:R
- C12, C8: value 20pF -> 22pF
- U2: value GD32F103C8T6 -> STM32F103C8T6
Connections:
- net GND: now also U2.8 (VSSA); no longer L1.1
- net PA11: now also R3.2; no longer R3.1
- net PA12: now also R2.2; no longer R2.1
- net USB_Data+: now also R2.1; no longer R2.2
- net USB_Data-: now also R3.1; no longer R3.2
- net VDD_3.3V: now also L1.1; no longer U2.9 (VDDA)
- net at L1.2: now also U2.9 (VDDA); no longer U2.8 (VSSA)
Other:
- note added: "STM32F103C8T6 最小系统"
- note removed: "GD32F103Cxxx 最小系统"
- moved on the sheet: C1, C10, C11, C3, C6, C8, J1, J2, L1
