File: UINIO-MCU-STM32F103C8T6.kicad_pcb (KiCad board)
At the start: 2 copper layers, 68.4 x 20.3 mm, 41 parts, among them J1 Conn_01x24_Pin, J2 Conn_01x24_Pin, J3 Conn_01x04_Pin, SW1 BOOT1, SW2 NRST, SW3 BOOT0, U1 ME6211C33M5G-N, U2 STM32F103C8T6, Y1 32.768KHz, Y2 8MHz

Commit message: Release UINIO-MCU-STM32F103C8T6 version 3.2.0.
Parts:
- moved R1 2.27 mm to (134.2, 95.7), turned to -90 degrees
- moved R12 0.50 mm to (134.7, 101.0)
- moved R11 0.39 mm to (132.2, 97.3)
Routing:
- net GND: track 135.3 -> 134.0 mm, vias 55 -> 59
